Commit message: Startup inter-robot calibration

File: ros2_ws/src/LIO-SAM_MID360_ROS2/config/robot.urdf.xacro (robot description, xacro)
@@ -2,33 +2,38 @@
 <robot name="lio" xmlns:xacro="http://tixiaoshan.github.io/">
   <xacro:property name="PI" value="3.1415926535897931" />
-  <link name="chassis_link"></link>
-  <link name="base_link"></link>
+  <!-- Namespace for frame names (default to empty string) -->
+  <xacro:arg name="namespace" default="" />
+  <!-- Create frame prefix with trailing slash if namespace is not empty -->
+  <xacro:property name="namespace_val" value="$(arg namespace)" />
+  <xacro:property name="frame_prefix" value="${namespace_val + '/' if namespace_val else ''}" />
+  <link name="${frame_prefix}chassis_link"></link>
+  <link name="${frame_prefix}base_link"></link>
   <joint name="base_link_joint" type="fixed">
-    <parent link="base_link"/>
-    <child link="chassis_link" />
+    <parent link="${frame_prefix}base_link"/>
+    <child link="${frame_prefix}chassis_link" />
     <origin xyz="0 0 0" rpy="0 0 0" />
   </joint>
-  <link name="livox_frame"> </link>
+  <link name="${frame_prefix}livox_frame"> </link>
   <joint name="lidar_joint" type="fixed">
-    <parent link="base_link" />
-    <child link="livox_frame" />
+    <parent link="${frame_prefix}base_link" />
+    <child link="${frame_prefix}livox_frame" />
     <origin xyz="0 0 0" rpy="0 0 0" />
   </joint>
-  <link name="imu_link"> </link>
+  <link name="${frame_prefix}imu_link"> </link>
   <joint name="imu_joint" type="fixed">
-    <parent link="chassis_link" />
-    <child link="imu_link" />
+    <parent link="${frame_prefix}chassis_link" />
+    <child link="${frame_prefix}imu_link" />
     <origin xyz="0 0 0" rpy="0 0 0" />
   </joint>
-  <link name="laser_sensor_frame"> </link>
+  <link name="${frame_prefix}laser_sensor_frame"> </link>
   <joint name="laser_joint" type="fixed">
-    <parent link="imu_link" />
-    <child link="laser_sensor_frame" />
+    <parent link="${frame_prefix}imu_link" />
+    <child link="${frame_prefix}laser_sensor_frame" />
     <origin xyz="0 0 0" rpy="0 0 0" />
   </joint>
-  <link name="navsat_link"> </link>
+  <link name="${frame_prefix}navsat_link"> </link>
   <joint name="navsat_joint" type="fixed">
-    <parent link="chassis_link" />
-    <child link="navsat_link" />
+    <parent link="${frame_prefix}chassis_link" />
+    <child link="${frame_prefix}navsat_link" />
     <origin xyz="0 0 0" rpy="0 0 0" />
   </joint>

Commit message: Add: only_rover_launch.py - launch file for rover without drone
And removed unused lio-sam frames

File: ros2_ws/src/LIO-SAM_MID360_ROS2/config/robot.urdf.xacro (robot description, xacro)
@@ -7,11 +7,5 @@
   <xacro:property name="namespace_val" value="$(arg namespace)" />
   <xacro:property name="frame_prefix" value="${namespace_val + '/' if namespace_val else ''}" />
-  <link name="${frame_prefix}chassis_link"></link>
   <link name="${frame_prefix}base_link"></link>
-  <joint name="base_link_joint" type="fixed">
-    <parent link="${frame_prefix}base_link"/>
-    <child link="${frame_prefix}chassis_link" />
-    <origin xyz="0 0 0" rpy="0 0 0" />
-  </joint>
   <link name="${frame_prefix}livox_frame"> </link>
   <joint name="lidar_joint" type="fixed">
@@ -20,21 +14,3 @@
     <origin xyz="0 0 0" rpy="0 0 0" />
   </joint>
-  <link name="${frame_prefix}imu_link"> </link>
-  <joint name="imu_joint" type="fixed">
-    <parent link="${frame_prefix}chassis_link" />
-    <child link="${frame_prefix}imu_link" />
-    <origin xyz="0 0 0" rpy="0 0 0" />
-  </joint>
-  <link name="${frame_prefix}laser_sensor_frame"> </link>
-  <joint name="laser_joint" type="fixed">
-    <parent link="${frame_prefix}imu_link" />
-    <child link="${frame_prefix}laser_sensor_frame" />
-    <origin xyz="0 0 0" rpy="0 0 0" />
-  </joint>
-  <link name="${frame_prefix}navsat_link"> </link>
-  <joint name="navsat_joint" type="fixed">
-    <parent link="${frame_prefix}chassis_link" />
-    <child link="${frame_prefix}navsat_link" />
-    <origin xyz="0 0 0" rpy="0 0 0" />
-  </joint>
 </robot>
